File: pcbr2/tach/tach.sch (KiCad schematic (older format))
At the start: 90 parts, among them J1 Screw_Terminal_01x02, J2 Conn_01x01, J3 Conn_01x01, J4 XF2M-1415-1A, J5 FTSH-105-01-L-DV-007-K, J6 Conn_01x01, J7 Conn_01x01, Q1 MMBT3904-7-F, Q2 MMBT3906-7-F, U1 TMP20AIDCK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

Commit message: this commit preserves the state of the repo as of 7/13/26. confirmed working in hardware.
Parts:
- removed D2: BAS40-04, TO_SOT_Packages_SMD:SOT-23, symbol Diode:BAS40-04
- removed Q2: MMBT3906-7-F, TO_SOT_Packages_SMD:SOT-23, symbol Device:Q_PNP_BEC
- removed RV1: 100k, Potentiometers:Potentiometer_Trimmer_Bourns_3224J, symbol Device:R_POT
- removed U2: TLV6001, TO_SOT_Packages_SMD:TSOT-23-5, symbol Amplifier_Operational:AD8603
- added C40: 0.1/10, Capacitors_SMD:C_0402, symbol Device:C
- added C41: 1.0/10, Capacitors_SMD:C_0402, symbol Device:C
- added C42: 0.01/10, Capacitors_SMD:C_0402, symbol Device:C
- added D2: SZMMBZ5222BLT1G, TO_SOT_Packages_SMD:SOT-23, symbol Device:D_Zener
- added R21: 18.2k 0.1%, Resistors_SMD:R_0402, symbol Device:R_US
- added U2: REF5025ADGK, Housings_SSOP:MSOP-8_3x3mm_Pitch0.65mm, symbol Reference_Voltage:REF5020ADGK
- C30: value 0.1/10 -> 1.0/10
- C36, C37: footprint Capacitors_SMD:C_0402 -> Capacitors_SMD:C_0805
- C4: value 0.1/16 -> 0.01/10
- H1, H2: footprint Mounting_Holes:MountingHole_2.5mm -> footprints:MountingHole_M3
- R1: value 22k -> 10k
- R2: value 100k -> 2.2k 0.1%; footprint Resistors_SMD:R_0402 -> Resistors_SMD:R_0805
- R5: value 100 -> 10k
- R8: value 10k -> 80.6k 0.1%
Connections:
- net +12V: now also R2.1, R8.1
- net +3.3VA: no longer C4.1, R1.1, R5.1
- net +3V3: now also C40.1, U2.2 (Vin)
- net COLD_JUNC: now also C4.1, R1.1; no longer U1.3 (Vout)
- net GND: now also C40.2, C41.2, C42.2, D2.2 (A), R21.2, U2.4 (GND); no longer R2.2
- net JNTRST: no longer J5.10 (Pin_10)
- net NRST: now also J5.10 (Pin_10)
- net OIL_TEMP: now also R5.1, D2.1 (K); no longer R8.1
- net OIL_TEMP_IN: now also R2.2, R5.2; no longer R8.2
- net STEPPER1: now also U6.31 (PA10); no longer U6.32 (PA11)
- net STEPPER2: now also U6.33 (PA12); no longer U6.31 (PA10)
- net STEPPER_EN: now also U6.32 (PA11); no longer U6.25 (PB12)
- net TACH: now also U6.16 (PA6); no longer U6.17 (PA7)
- net BATT_SENS: now reaches U6.10 (PA0)
- net BATT_SENS: now also R8.2, C42.1, R21.1
- net 2V5_REF: now reaches U6.14 (PA4)
- net 2V5_REF: now also U2.6 (Vout)
- net at R1.2: now also U1.3 (Vout); no longer R2.1
- new net: C41.1, U2.5 (Trim/NR)
Other:
- note added: "For use with grounded-tip thermocouples, e.g. spark plug gasket mount.\nDual-supply moves common mode range below ground to provide noise\nrejection for noise caused by ground difference from tach supply to engine case."
- note added: "Optional voltage reference. No external Vref pin,\nso we just use it as a cal value.\n\nERRATUM: needs output cap, 1-50uF (tested 10uF, doesn't work without)"
- note added: "We're already measuring voltage, so we'll use that measurement to \nback out the effect from battery voltage variation."
- note removed: "Changelist:\nLarger holes for wires\nUse 2x5 Samtec 0.5" header ARM standard JTAG\nFull input protection e.g. X310\nReview and fix mounting hole spacing/dia\nLarger heatsink pad for regulators\nReview ADC pins"
- note removed: "For use with grounded-tip thermocouples, e.g. spark plug gasket mount.\nDual-supply moves common mode range below ground to provide noise\nrejection for noise caused by ground difference from tach supply to engine case.\nThe protection diodes effectively limit the common-mode to [-0.35V, 0.35V].\nThis should be OK -- but transient noise pickup from the spark plug wires\ncould cause CM to move out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"
- note removed: "Oil temp is a VDO resistance sensor with a grounded body."
- note removed: "This isn't a great overvoltage protection circuit.\nHow do you protect without adding series R?"
- note removed: "Trim for 5mA or calibrate \nto around 1.5V at 100C"
- moved on the sheet: C1, C5, J3
